File: Game_Cat_R4.kicad_pcb (KiCad board)
At the start: 2 copper layers, 160 x 60 mm, 194 parts, among them J1 USB_C, J2 CAN, J3 Joystick, J4 Micro_SD, J5 CORTEX-SWD, J6 UART, J7 PWM, Q1 2N2907, Q10 2N7002, Q2 2N2907, Q3 2N7002, Q4 DMP3056L, Q5 NTR1P02LT1, Q6 BS138, Q7 BS138, Q8 BS138, Q9 BS138, SW1 A, SW2 B, SW3 X, SW4 Y, SW5 L, SW6 R, SW7 Reset, SW8 SW_SPDT, U1 ATSAMD21G18A, U10 LM61, U11 MCP73831, U12 TPS54231, U2 TPD2E2U06, U3 MCP2518FD, U4 MCP2562FD, U5 24LC512, U6 23KXX, U7 74HC4051, U8 MMA8452Q, U9 SST26VF032B, Y1 20Mhz, Y3 ABS25

Commit message: 08/06/24/A
Parts:
- removed Y3: ABS25, x_Crystal:Crystal_SMD_ABS25_4Pin_8.0x3.8mm
- added Y2: Crystal_GND3, x_Crystal:MS1V-T1K_32.768KHZ_7PF_20PPM_TA, F.Cu at (117.6, 94.5)
- moved C9 4.25 mm to (120.2, 91.3)
- moved C8 0.73 mm to (120.2, 97.7)
Routing:
- net Net-(U1-PA00/XIN32): track 15.4 -> 11.2 mm

Commit message: 25/01/24/A
Parts:
- removed R26: 10K, Resistor_SMD:R_1206_3216Metric
- added D10: BAT60J, Diode_SMD:D_SOD-323_HandSoldering, F.Cu at (100.1, 85.9)
- added R63: 0R, Resistor_SMD:R_1206_3216Metric, F.Cu at (100.6, 97.7)
- added R64: 0R, Resistor_SMD:R_1206_3216Metric, B.Cu at (171.4, 112.9)
- C12: value 10uF -> 1uF
- C36: value 4.7uF -> 1uF
- F1: footprint x_Fuses:MF-SMDF200-2 -> x_Fuses:MF_SMDF200
- R37: value 68K -> 30K
- R4: value 1K -> 10K
- R40: value 1K -> 180
- R43: value 68K -> 3K
- U5: footprint Package_SO:SOIC-8_3.9x4.9mm_P1.27mm -> Package_SO:SOIC-8W_5.3x5.3mm_P1.27mm
- U9: footprint Package_SO:SOIJ-8_5.3x5.3mm_P1.27mm -> Package_SO:SOIC-8W_5.3x5.3mm_P1.27mm
- moved R4 37.6 mm to (82.1, 119.2), turned to 180 degrees
- moved R9 4.98 mm to (82.1, 123.9)
- moved TP21 2.74 mm to (96.3, 95.6)
- moved U5 1.17 mm to (139.8, 113.4)
- moved D13 0.78 mm to (73.9, 122.5)
- moved R19 0.78 mm to (69.6, 122.5)
- moved R56 0.43 mm to (82.1, 121.5)
- moved TP16 0.36 mm to (86.2, 121.5)
- moved Q3 0.36 mm to (77.9, 117.8)
- moved R18 0.26 mm to (82.1, 116.8)
- moved D12 0.26 mm to (73.9, 118.7)
- moved R8 0.26 mm to (69.6, 118.7)
- moved TP15 0.16 mm to (86.2, 116.8)
- moved Q10 0.15 mm to (77.9, 122.5)
- moved TP23 0.10 mm to (142.0, 103.1)
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Connections:
- C3 pad 2: /USB COMMUNICATIONS/OSC1 -> /USB COMMUNICATIONS/OSC2
- C4 pad 2: /USB COMMUNICATIONS/OSC2 -> /USB COMMUNICATIONS/OSC1
- C42 pad 1: +3V3 -> Net-(C42-Pad1)
- L1 pad 1: +3V3 -> Net-(L1-Pad1)
- L3 pad 2: +3V3 -> Net-(C42-Pad1)
- Q10 pad 2: Net-(D13-K) -> GND
- Q10 pad 3: GND -> Net-(D13-K)
- Q3 pad 2: Net-(D12-K) -> GND
- Q3 pad 3: GND -> Net-(D12-K)
- R4 pad 1: SWDCLK -> GND
- R4 pad 2: +3V3 -> Net-(Q3-G)
- R42 pad 1: +3V3 -> Net-(C42-Pad1)
- R9 pad 2: Net-(Q3-G) -> Net-(Q10-G)
- SW1 pad 1: unconnected-(SW1-Pad1) -> /JOYSTICK, BUTTONS & SENSES/Button_A
- SW1 pad 2: /JOYSTICK, BUTTONS & SENSES/Button_A -> unconnected-(SW1-Pad2)
- SW2 pad 3: /JOYSTICK, BUTTONS & SENSES/Button_B -> unconnected-(SW2-Pad3)
- SW2 pad 4: unconnected-(SW2-Pad4) -> /JOYSTICK, BUTTONS & SENSES/Button_B
- SW3 pad 3: unconnected-(SW3-Pad3) -> /JOYSTICK, BUTTONS & SENSES/Button_X
- SW3 pad 4: /JOYSTICK, BUTTONS & SENSES/Button_X -> unconnected-(SW3-Pad4)
- SW4 pad 3: unconnected-(SW4-Pad3) -> /JOYSTICK, BUTTONS & SENSES/Button_Y
- SW4 pad 4: /JOYSTICK, BUTTONS & SENSES/Button_Y -> unconnected-(SW4-Pad4)
- U1 pad 25: SCL -> SDA
- U1 pad 26: SDA -> SCL
- Y1 pad 1: /USB COMMUNICATIONS/OSC2 -> /USB COMMUNICATIONS/OSC1
- Y1 pad 2: /USB COMMUNICATIONS/OSC1 -> /USB COMMUNICATIONS/OSC2
Routing:
- net +3V3: track 593.6 -> 577.1 mm
- net GND: track 64.9 -> 55.5 mm, vias 88 -> 94
- net Net-(C42-Pad1): track 0.00 -> 8.97 mm
- net /USB COMMUNICATIONS/OSC2: track 17.2 -> 22.3 mm
- net /USB COMMUNICATIONS/OSC1: track 15.8 -> 20.6 mm
- net Net-(L1-Pad1): track 0.00 -> 3.08 mm
- net RESET: track 123.0 -> 125.6 mm
- net SWDCLK: track 88.5 -> 86.0 mm
- net Net-(D13-K): track 2.08 -> 3.41 mm
- net CAN_SS: track 21.2 -> 20.3 mm
- net CAN_MISO: track 22.9 -> 23.7 mm
- net /USB COMMUNICATIONS/TXCAN: track 20.2 -> 19.5 mm
- net VAA: track 126.4 -> 125.8 mm
- net Net-(D12-K): track 3.57 -> 3.02 mm
- net CAN_INT: track 17.8 -> 17.3 mm
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Other:
- board text added: "Game//Cat R4 Version 4.2.2 Copyrigth 2025 Designed in Colombia"
- board text removed: "Game//Cat Version 4.1.4 Copyrigth 2022 Designed in Colombia"

Commit message: 25/01/24/C
Other:
- board text added: "[Off-On]"
- board text removed: "On-Off"
Changed lines of the file:
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@@
 		)
 	)
-	(gr_text "On-Off"
-		(at 187.706 77.724 -20)
+	(gr_text "[Off-On]"
+		(at 187.706 77.724 340)
 		(layer "F.SilkS")
 		(effects

Commit message: 25/01/26/A
Parts:
- removed D7: BAT60J, Diode_SMD:D_SOD-323_HandSoldering
- moved C44 2.42 mm to (171.8, 83.5)
- moved C42 0.87 mm to (171.4, 107.7)
- moved L3 0.86 mm to (177.6, 108.0)
- moved R42 0.86 mm to (174.1, 107.7)
- moved R64 0.46 mm to (171.4, 113.3)
Routing:
- net /POWER SUPPLY/M: track 16.0 -> 13.6 mm
- net Net-(D6-K): track 7.54 -> 6.13 mm
- net Net-(U12-FB): track 19.1 -> 19.9 mm
