File: Game_Cat_R4.kicad_pcb (KiCad board)
At the start: 2 copper layers, 160 x 60 mm, 195 parts, among them J1 USB_C, J2 CAN, J3 Joystick, J4 Micro_SD, J5 CORTEX-SWD, J6 UART, J7 PWM, Q1 2N2907, Q10 2N7002, Q2 2N2907, Q3 2N7002, Q4 DMP3056L, Q5 NTR1P02LT1, Q6 BS138, Q7 BS138, Q8 BS138, Q9 BS138, SW1 A, SW2 B, SW3 X, SW4 Y, SW5 L, SW6 R, SW7 Reset, SW8 SW_SPDT, U1 ATSAMD21G18A, U10 LM61, U11 MCP73831, U12 TPS54231, U2 TPD2E2U06, U3 MCP2518FD, U4 MCP2562FD, U5 24LC512, U6 23KXX, U7 74HC4051, U8 MMA8452Q, U9 SST26VF032B, Y1 20Mhz, Y2 Crystal_GND3

Commit message: 05/25/25/A
Parts:
- removed J4: Micro_SD, x_Connector_Card:MICRO_SD_HC_DM3AT
- removed U4: MCP2562FD, Package_SO:SOIC-8_3.9x4.9mm_P1.27mm
- added J8: DM3AT-SF-PEJM5, x_Connector_Card:DM3AT_SF_PEJM5, F.Cu at (98.9, 121.3)
- added U13: TCAN337GDR, Package_SO:SOIC-8_3.9x4.9mm_P1.27mm, F.Cu at (144.6, 82.5)
- Q4: value DMP3056L -> FDN340P
- U5, U9: footprint Package_SO:SOIC-8W_5.3x5.3mm_P1.27mm -> Package_SO:SOIC-8_5.3x5.3mm_P1.27mm
- moved C31 0.18 mm to (97.5, 111.1)
Routing:
- net SPI_MISO: track 61.6 -> 70.1 mm
- net VAA: track 125.8 -> 124.1 mm, vias 6 -> 5
- net +3V3: track 576.7 -> 575.1 mm
- net SPI_MOSI: track 56.2 -> 56.8 mm
- net SPI_SCK: track 63.2 -> 63.8 mm
- net GND: vias 94 -> 92

Commit message: 03/11/26/Update BOM & Models VRML
Parts:
- BT1: footprint x_Connector_JST:Connector_1x02_P2.0mm -> x_Connector_JST:S2B_PH_SM4_TB
- SW1: footprint x_Button_Switch_SMD:SW_PUSH_SMD_125x12mm_SNAP_GREEN -> x_Button_Switch_SMD:SWITCH_TACTILE_SPST_PLUNGER_CAP_GREEN_12x12mm_SMD
- SW2: footprint x_Button_Switch_SMD:SW_PUSH_SMD_125x12mm_SNAP_RED -> x_Button_Switch_SMD:SWITCH_TACTILE_SPST_PLUNGER_CAP_RED_12x12mm_SMD
- SW3: footprint x_Button_Switch_SMD:SW_PUSH_SMD_125x12mm_SNAP_BLUE -> x_Button_Switch_SMD:SWITCH_TACTILE_SPST_PLUNGER_CAP_BLUE_12x12mm_SMD
- SW4: footprint x_Button_Switch_SMD:SW_PUSH_SMD_125x12mm_SNAP_YELLOW -> x_Button_Switch_SMD:SWITCH_TACTILE_SPST_PLUNGER_CAP_YELLOW_12x12mm_SMD
- Y2: footprint x_Crystal:MS1V-T1K_32.768KHZ_7PF_20PPM_TA -> x_Crystal:MS1V_T1K_32.768KHZ_7PF_20PPM_TA
- moved R30 2.41 mm to (97.7, 86.1)
- moved R31 2.39 mm to (95.3, 86.1)
- moved TP12 1.32 mm to (161.9, 88.3)
- moved D13 0.94 mm to (73.9, 123.4)
- moved R19 0.94 mm to (69.6, 123.4)
- moved TP21 0.20 mm to (96.3, 95.8)
- moved C31 0.08 mm to (97.5, 111.0)
Routing:
- net SPI_MISO: track 70.1 -> 61.2 mm
- net SWDCLK: track 86.0 -> 91.4 mm
- net Net-(J5-Pin_4): track 14.1 -> 18.8 mm
- net Net-(C10-Pad1): track 14.8 -> 18.9 mm
- net /USB COMMUNICATIONS/VBUS: track 25.9 -> 21.9 mm
- net USD_CK: track 60.0 -> 63.7 mm
- net SPI_MOSI: track 56.8 -> 53.7 mm
- net VCC: track 46.8 -> 44.9 mm
- net SPI_SCK: track 63.8 -> 62.1 mm
- net +3V3: track 575.1 -> 573.9 mm
- net SWDIO: track 91.5 -> 90.7 mm
- net RESET: track 125.6 -> 124.9 mm
- net GND: vias 92 -> 89
Other:
- rule pad_to_mask_clearance: 0.0508 -> 0

Commit message: 03/12/26/Update BOM & Models VRML
Parts:
- BZ1: footprint Buzzer_Beeper:Buzzer_12x9.5RM7.6 -> x_Buzzer:AT_1224_TWT_5V_2_R
- C1: value 10uF -> 4.7uF
- D1, D12, D13, D2, D4, D5: footprint LED_SMD:LED_0805_2012Metric_Castellated -> LED_SMD:LED_0805_2012Metric
- F1: value 500mA -> 2016L100PR
- L1: value BLM18PG471 -> FB321611T
- Q1, Q2: value 2N2907 -> MMBT2907A
- Q6, Q7, Q8, Q9: value BS138 -> BSS138
- U10: value LM61 -> TC1046
- U3: value MCP2518FD -> MCP2518FDT
- U5: value 24LC512 -> 24CSM01
- U6: value 23KXX -> 23K256
- U9: value SST26VF032B -> AT25DF641A
- Y1: value 20Mhz -> 4Mhz
- moved BZ1 3.25 mm to (67.7, 80.0), turned to 0 degrees
Routing:
- net Net-(BZ1-+): track 9.03 -> 7.96 mm
