File: Game_Cat_R4.kicad_sch (KiCad schematic)
At the start: 0 parts

Commit message: 25/01/24/C
Other:
- note added: "JOYSTCK BUTTONS & SENSES"
- note added: "MICRO CONTROLLER"
- note removed: "JOYSTCK- BUTTONS & SENSES"
- note removed: "MICRO- CONTROLLER"
