File: joystick_buttons_senses.kicad_sch (KiCad schematic)
At the start: 73 parts, among them J3 Joystick, J4 Micro_SD, Q1 2N2907, Q2 2N2907, SW1 A, SW2 B, SW3 X, SW4 Y, SW5 L, SW6 R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

Commit message: 25/01/24/A
Parts:
- U5: footprint Package_SO:SOIC-8_3.9x4.9mm_P1.27mm -> Package_SO:SOIC-8W_5.3x5.3mm_P1.27mm
- U9: footprint Package_SO:SOIJ-8_5.3x5.3mm_P1.27mm -> Package_SO:SOIC-8W_5.3x5.3mm_P1.27mm
Connections:
- net Button_A: now also SW1.1; no longer SW1.2
- net Button_B: now also SW2.4; no longer SW2.3
- net Button_X: now also SW3.3; no longer SW3.4
- net Button_Y: now also SW4.3; no longer SW4.4
Changed lines of the file:
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@@
 	)
 	(no_connect
-		(at 35.56 59.69)
+		(at 35.56 62.23)
 	)
 	(no_connect
@@
 	)
 	(no_connect
-		(at 35.56 68.58)
+		(at 35.56 71.12)
 	)
 	(no_connect
-		(at 35.56 41.91)
+		(at 35.56 44.45)
 	)
 	(no_connect
-		(at 35.56 53.34)
+		(at 35.56 50.8)
 	)
 	(no_connect
@@
 	(wire
 		(pts
-			(xy 36.83 41.91) (xy 48.26 41.91)
-		)
-		(stroke
-			(width 0)
-			(type default)
-		)
-	)
-	(wire
-		(pts
 			(xy 22.86 59.69) (xy 22.86 62.23)
 		)
@@
 	(wire
 		(pts
-			(xy 35.56 62.23) (xy 36.83 62.23)
+			(xy 35.56 59.69) (xy 60.96 59.69)
 		)
 		(stroke
@@
 	(wire
 		(pts
-			(xy 36.83 71.12) (xy 36.83 68.58)
-		)
-		(stroke
-			(width 0)
-			(type default)
-		)
-	)
-	(wire
-		(pts
 			(xy 25.4 50.8) (xy 22.86 50.8)
 		)
@@
 	(wire
 		(pts
-			(xy 36.83 68.58) (xy 67.31 68.58)
-		)
-		(stroke
-			(width 0)
-			(type default)
-		)
-	)
-	(wire
-		(pts
 			(xy 93.98 128.27) (xy 93.98 129.54)
 		)
@@
 	(wire
 		(pts
-			(xy 35.56 50.8) (xy 54.61 50.8)
+			(xy 35.56 53.34) (xy 54.61 53.34)
 		)
 		(stroke
@@
 	(wire
 		(pts
-			(xy 35.56 44.45) (xy 36.83 44.45)
+			(xy 35.56 41.91) (xy 48.26 41.91)
 		)
 		(stroke
@@
 	(wire
 		(pts
-			(xy 36.83 62.23) (xy 36.83 59.69)
-		)
-		(stroke
-			(width 0)
-			(type default)
-		)
-	)
-	(wire
-		(pts
 			(xy 222.25 39.37) (xy 222.25 41.91)
 		)
@@
 	(wire
 		(pts
-			(xy 35.56 71.12) (xy 36.83 71.12)
+			(xy 35.56 68.58) (xy 67.31 68.58)
 		)
 		(stroke
@@
 	(wire
 		(pts
-			(xy 36.83 59.69) (xy 60.96 59.69)
-		)
-		(stroke
-			(width 0)
-			(type default)
-		)
-	)
-	(wire
-		(pts
 			(xy 99.06 165.1) (xy 99.06 166.37)
 		)
@@
 	(wire
 		(pts
-			(xy 36.83 44.45) (xy 36.83 41.91)
-		)
-		(stroke
-			(width 0)
-			(type default)
-		)
-	)
-	(wire
-		(pts
 			(xy 167.64 55.88) (xy 187.96 55.88)
 		)
@@
 	(wire
 		(pts
-			(xy 54.61 41.91) (xy 54.61 50.8)
+			(xy 54.61 41.91) (xy 54.61 53.34)
 		)
 		(stroke
@@
 	)
 	(label "Button_B"
-		(at 38.1 50.8 0)
+		(at 38.1 53.34 0)
 		(fields_autoplaced yes)
 		(effects
@@
 			)
 		)
-		(property "Footprint" "Package_SO:SOIC-8_3.9x4.9mm_P1.27mm"
+		(property "Footprint" "Package_SO:SOIC-8W_5.3x5.3mm_P1.27mm"
 			(at 39.37 123.19 0)
 			(effects
@@
 			)
 		)
-		(property "Footprint" "Package_SO:SOIJ-8_5.3x5.3mm_P1.27mm"
+		(property "Footprint" "Package_SO:SOIC-8W_5.3x5.3mm_P1.27mm"
 			(at 113.03 187.96 0)
 			(effects

Commit message: 05/25/25/A
Parts:
- removed J4: Micro_SD, x_Connector_Card:MICRO_SD_HC_DM3AT, symbol Connector:Micro_SD_Card_Det
- added J8: DM3AT-SF-PEJM5, x_Connector_Card:DM3AT_SF_PEJM5, symbol x_Connectors:DM3AT-SF-PEJM5
- U5, U9: footprint Package_SO:SOIC-8W_5.3x5.3mm_P1.27mm -> Package_SO:SOIC-8_5.3x5.3mm_P1.27mm
Connections:
- net +3V3: now also J8.4 (VDD)
- net GND: now also J8.6 (VSS), J8.P1 (SHIELD), J8.P2 (SHIELD__1), J8.P3 (SHIELD__2), J8.P4 (SHIELD__3), J8.SWB (A)
- net SPI_MISO: now also J8.7 (DAT0)
- net SPI_MOSI: now also J8.3 (CMD)
- net SPI_SCK: now also J8.5 (CLK)
- net USD_CK: now also J8.SWA (B)
- net USD_SS: now also J8.2 (CD/DAT3)
Other:
- moved on the sheet: BZ1, C30, Q1, R25, R27, R59, TP10, TP20, TP9

Commit message: 03/11/26/Update BOM & Models VRML
Parts:
- C16, C17, C18, C19, C24: Digikey (none) -> C3216X7R2E104K160AE
- C20, C26, C27, C31: Digikey (none) -> GRM21A5C2E100JW01D
- C22: Digikey (none) -> C0805C220J5GAC7800
- C23, C25, C28, C30: Digikey (none) -> GRM3195C1H113JA01D
- J3: footprint x_Button_Switch_THT:TUMB_JOYSTICK -> x_Joystick:JOYSTICK_TUMB; Digikey (none) -> 09032
- J8: Digikey (none) -> DM3AT-SF-PEJM5; MANUFACTURER Hirose Electric Co Ltd -> (none); MAXIMUM_PACKAGE_HEIGHT 1.83 mm -> (none); PARTREV 20200913 -> (none); STANDARD Manufacturer Recommendations -> (none)
- R10, R11, R12, R13, R14, R15, R16, R17, R20, R21, R25, R29, R5, R54, R57, R58, R59, R7: Digikey (none) -> RC1206FR-0710KL
- R23: Digikey (none) -> RC1206FR-07100KL
- R24: Digikey (none) -> RC1206JR-0733RL
- R27: Digikey (none) -> RC1206FR-072K2L
- R28: Digikey (none) -> RC1206FR-0710RL
- R55: Digikey (none) -> RC1206FR-074K7L
- SW1: footprint x_Button_Switch_SMD:SW_PUSH_SMD_125x12mm_SNAP_GREEN -> x_Button_Switch_SMD:SWITCH_TACTILE_SPST_PLUNGER_CAP_GREEN_12x12mm_SMD
- SW2: footprint x_Button_Switch_SMD:SW_PUSH_SMD_125x12mm_SNAP_RED -> x_Button_Switch_SMD:SWITCH_TACTILE_SPST_PLUNGER_CAP_RED_12x12mm_SMD
- SW3: footprint x_Button_Switch_SMD:SW_PUSH_SMD_125x12mm_SNAP_BLUE -> x_Button_Switch_SMD:SWITCH_TACTILE_SPST_PLUNGER_CAP_BLUE_12x12mm_SMD
- SW4: footprint x_Button_Switch_SMD:SW_PUSH_SMD_125x12mm_SNAP_YELLOW -> x_Button_Switch_SMD:SWITCH_TACTILE_SPST_PLUNGER_CAP_YELLOW_12x12mm_SMD
- SW5, SW6: Digikey (none) -> CT1102V3.85F160
- TP10, TP17, TP18, TP19, TP2, TP20, TP21, TP22, TP27, TP28, TP3, TP4, TP5, TP6, TP7, TP8, TP9: now not fitted
- U10: value LM61 -> TC1046; Digikey (none) -> TC1046VNBTR
- U5: value 24LC512 -> 24CSM01; Digikey (none) -> 24CSM01T-E/ST
- U6: value 23KXX -> 23K256; Digikey (none) -> 23K256-I/SN
- U7: Digikey (none) -> CD74HC4051QM96Q1
- U8: Digikey (none) -> MMA8452QT
- U9: value SST26VF032B -> AT25DF641A; Digikey (none) -> AT25DF641A-SH-B

Commit message: 03/12/26/Update BOM & Models VRML
Parts:
- BZ1: footprint Buzzer_Beeper:Buzzer_12x9.5RM7.6 -> x_Buzzer:AT_1224_TWT_5V_2_R; Digikey (none) -> AI-1223-TWT-3V-2-R
- LCD1: Digikey (none) -> SSW-108-01-F-S
- Q1, Q2: value 2N2907 -> MMBT2907A; Digikey (none) -> MMBT2907A-7-F
- R22: Digikey (none) -> N5AC501085
- SW1, SW2, SW3, SW4: Digikey (none) -> TL3300AF160Q
Changed lines of the file:
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@@
 			)
 		)
-		(property "Datasheet" "~"
+		(property "Datasheet" "https://www.farnell.com/datasheets/1580320.pdf"
 			(at 158.75 102.87 0)
 			(effects
@@
 			)
 		)
-		(property "Description" ""
+		(property "Description" "CDS PHOTORESISTOR 100KOHM TO-18"
+			(at 158.75 101.6 0)
+			(effects
+				(font
+					(size 1.27 1.27)
+				)
+				(hide yes)
+			)
+		)
+		(property "Digikey" "N5AC501085"
 			(at 158.75 101.6 0)
 			(effects
@@
 	)
 	(symbol
-		(lib_id "Device:Buzzer")
-		(at 248.92 88.9 0)
-		(unit 1)
-		(exclude_from_sim no)
-		(in_bom yes)
-		(on_board yes)
-		(dnp no)
-		(property "Reference" "BZ1"
-			(at 252.7808 88.1634 0)
-			(effects
-				(font
-					(size 1.27 1.27)
-				)
-				(justify left)
-			)
-		)
-		(property "Value" "Buzzer"
-			(at 252.7808 90.4748 0)
-			(effects
-				(font
-					(size 1.27 1.27)
-				)
-				(justify left)
-			)
-		)
-		(property "Footprint" "Buzzer_Beeper:Buzzer_12x9.5RM7.6"
-			(at 248.285 86.36 90)
-			(effects
-				(font
-					(size 1.27 1.27)
-				)
-				(hide yes)
-			)
-		)
-		(property "Datasheet" "~"
-			(at 248.285 86.36 90)
-			(effects
-				(font
-					(size 1.27 1.27)
-				)
-				(hide yes)
-			)
-		)
-		(property "Description" ""
-			(at 248.92 88.9 0)
-			(effects
-				(font
-					(size 1.27 1.27)
-				)
-				(hide yes)
-			)
-		)
-		(pin "1"
-		)
-		(pin "2"
-		)
-		(instances
-			(project "Game_Cat_R4"
-				(path "/96315415-cfed-47d2-b3dd-d782358bd0df/00000000-0000-0000-0000-00005ce8b424"
-					(reference "BZ1")
-					(unit 1)
-				)
-			)
-		)
-	)
-	(symbol
 		(lib_id "Device:Q_PNP_BEC")
 		(at 241.3 99.06 0)
@@
 			)
 		)
-		(property "Value" "2N2907"
+		(property "Value" "MMBT2907A"
 			(at 246.126 100.203 0)
 			(effects
@@
 			)
 		)
-		(property "Datasheet" "~"
+		(property "Datasheet" "https://mm.digikey.com/Volume0/opasdata/d220001/medias/docus/900/MMBT2907A_Rev2016.pdf"
 			(at 241.3 99.06 0)
 			(effects
@@
 			)
 		)
+		(property "Digikey" "MMBT2907A-7-F"
+			(at 241.3 99.06 0)
+			(effects
+				(font
+					(size 1.27 1.27)
+				)
+				(hide yes)
+			)
+		)
 		(pin "1"
 		)
@@
 			)
 		)
-		(property "Value" "2N2907"
-			(at 247.8786 48.133 0)
+		(property "Value" "MMBT2907A"
+			(at 263.144 51.562 0)
 			(effects
 				(font
@@
 			)
 		)
-		(property "Datasheet" "~"
+		(property "Datasheet" "https://mm.digikey.com/Volume0/opasdata/d220001/medias/docus/900/MMBT2907A_Rev2016.pdf"
 			(at 252.73 46.99 0)
 			(effects
@@
 			)
 		)
+		(property "Digikey" "MMBT2907A-7-F"
+			(at 252.73 46.99 0)
+			(effects
+				(font
+					(size 1.27 1.27)
+				)
+				(hide yes)
+			)
+		)
 		(pin "1"
 		)
@@
 			)
 		)
-		(property "Datasheet" ""
+		(property "Datasheet" "https://mm.digikey.com/Volume0/opasdata/d220001/medias/docus/6129/ssw-1xx-xx-xxx-x-xx-xxx-xx-mkt.pdf"
 			(at 229.87 25.4 0)
 			(effects
@@
 					(size 3.048 3.048)
 				)
+				(hide yes)
+			)
+		)
+		(property "Description" "CONN RCPT 8POS 0.1 GOLD PCB"
+			(at 229.87 25.4 0)
+			(effects
+				(font
+					(size 1.27 1.27)
+				)
+				(hide yes)
 			)
 		)
-		(property "Description" ""
+		(property "Digikey" "SSW-108-01-F-S"
 			(at 229.87 25.4 0)
 			(effects
@@
 					(size 1.524 1.524)
 				)
+				(hide yes)
 			)
 		)
@@
 			)
 		)
-		(property "Datasheet" ""
+		(property "Datasheet" "https://configured-product-images.s3.amazonaws.com/Datasheets/TL3300.pdf"
 			(at 30.48 43.18 0)
 			(effects
@@
 					(size 1.524 1.524)
 				)
+				(hide yes)
 			)
 		)
@@
 			)
 		)
+		(property "Digikey" "TL3300AF160Q"
+			(at 30.48 41.91 0)
+			(effects
+				(font
+					(size 1.27 1.27)
+				)
+				(hide yes)
+			)
+		)
 		(pin "1"
 		)
@@
 			)
 		)
-		(property "Datasheet" ""
+		(property "Datasheet" "https://configured-product-images.s3.amazonaws.com/Datasheets/TL3300.pdf"
 			(at 30.48 52.07 0)
 			(effects
@@
 					(size 1.524 1.524)
 				)
+				(hide yes)
 			)
 		)
@@
 			)
 		)
+		(property "Digikey" "TL3300AF160Q"
+			(at 30.48 50.8 0)
+			(effects
+				(font
+					(size 1.27 1.27)
+				)
+				(hide yes)
+			)
+		)
 		(pin "1"
 		)
@@
 			)
 		)
-		(property "Datasheet" ""
+		(property "Datasheet" "https://configured-product-images.s3.amazonaws.com/Datasheets/TL3300.pdf"
 			(at 30.48 60.96 0)
 			(effects
@@
 					(size 1.524 1.524)
 				)
+				(hide yes)
 			)
 		)
@@
 			)
 		)
+		(property "Digikey" "TL3300AF160Q"
+			(at 30.48 59.69 0)
+			(effects
+				(font
+					(size 1.27 1.27)
+				)
+				(hide yes)
+			)
+		)
 		(pin "1"
 		)
@@
 			)
 		)
-		(property "Datasheet" ""
+		(property "Datasheet" "https://configured-product-images.s3.amazonaws.com/Datasheets/TL3300.pdf"
 			(at 30.48 69.85 0)
 			(effects
@@
 					(size 1.524 1.524)
 				)
+				(hide yes)
 			)
 		)
@@
 			)
 		)
+		(property "Digikey" "TL3300AF160Q"
+			(at 30.48 68.58 0)
+			(effects
+				(font
+					(size 1.27 1.27)
+				)
+				(hide yes)
+			)
+		)
 		(pin "1"
 		)
@@
 					(unit 1)
 				)
+			)
+		)
+	)
+	(symbol
+		(lib_id "Device:Buzzer")
+		(at 248.92 88.9 0)
+		(unit 1)
+		(exclude_from_sim no)
+		(in_bom yes)
+		(on_board yes)
+		(dnp no)
+		(fields_autoplaced yes)
+		(property "Reference" "BZ1"
+			(at 253.365 87.63 0)
+			(effects
+				(font
+					(size 1.27 1.27)
+				)
+				(justify left)
+			)
+		)
+		(property "Value" "Buzzer"
+			(at 253.365 90.17 0)
+			(effects
+				(font
+					(size 1.27 1.27)
+				)
+				(justify left)
+			)
+		)
+		(property "Footprint" "x_Buzzer:AT_1224_TWT_5V_2_R"
+			(at 248.285 86.36 90)
+			(effects
+				(font
+					(size 1.27 1.27)
+				)
+				(hide yes)
+			)
+		)
+		(property "Datasheet" "https://puiaudio.com/file/specs-AI-1223-TWT-3V-2-R.pdf"
+			(at 248.285 86.36 90)
+			(effects
+				(font
+					(size 1.27 1.27)
+				)
+				(hide yes)
+			)
+		)
+		(property "Description" "BUZZER MAGNETIC 3V 12MM TH"
+			(at 248.92 88.9 0)
+			(effects
+				(font
+					(size 1.27 1.27)
+				)
+				(hide yes)
+			)
+		)
+		(property "Digikey" "AI-1223-TWT-3V-2-R"
+			(at 248.92 88.9 0)
+			(effects
+				(font
+					(size 1.27 1.27)
+				)
+				(hide yes)
+			)
+		)
+		(pin "1"
+		)
+		(pin "2"
+		)
+		(instances
+			(project "Game_Cat_R4"
+				(path "/96315415-cfed-47d2-b3dd-d782358bd0df/00000000-0000-0000-0000-00005ce8b424"
+					(reference "BZ1")
+					(unit 1)
+				)
