File: microcontroller.kicad_sch (KiCad schematic)
At the start: 10 parts, among them U1 ATSAMD21G18A, Y2 32Khz

Commit message: 26/12/13/A
Parts:
- removed Y2: 32Khz, Crystal:Crystal_SMD_MicroCrystal_MS1V-T1K, symbol Device:Crystal
- added Y3: ABS25, x_Crystal:Crystal_SMD_Abracon_ABS25-4Pin_8.0x3.8mm, symbol Device:Crystal_GND24
Connections:
- net at C9.2, U1.1 (PA00/XIN32): now also Y3.1
- net at C8.2, U1.2 (PA01/XOUT32): now also Y3.4
- no-connect marks 0 -> 2
Changed lines of the file:
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@@
   (junction (at 101.6 52.07) (diameter 0) (color 0 0 0 0)
   )
+  (no_connect (at 106.68 58.42))
+  (no_connect (at 96.52 58.42))
   (wire (pts (xy 101.6 64.77) (xy 100.33 64.77))
     (stroke (width 0) (type default))
@@
     (stroke (width 0) (type default))
   )
-  (wire (pts (xy 106.68 52.07) (xy 101.6 52.07))
+  (wire (pts (xy 110.49 52.07) (xy 101.6 52.07))
     (stroke (width 0) (type default))
   )
@@
     (stroke (width 0) (type default))
   )
-  (wire (pts (xy 106.68 52.07) (xy 106.68 78.74))
+  (wire (pts (xy 110.49 52.07) (xy 110.49 78.74))
     (stroke (width 0) (type default))
   )
@@
     (stroke (width 0) (type default))
   )
-  (wire (pts (xy 106.68 78.74) (xy 115.57 78.74))
+  (wire (pts (xy 110.49 78.74) (xy 115.57 78.74))
     (stroke (width 0) (type default))
   )
@@
     )
   )
-  (symbol (lib_id "Device:Crystal") (at 101.6 58.42 90) (mirror x) (unit 1)
-    (in_bom yes) (on_board yes) (dnp no)
-    (property "Reference" "Y2" (at 98.2726 57.2516 90)
-      (effects (font (size 1.27 1.27)) (justify left))
-    )
-    (property "Value" "32Khz" (at 98.2726 59.563 90)
-      (effects (font (size 1.27 1.27)) (justify left))
-    )
-    (property "Footprint" "Crystal:Crystal_SMD_MicroCrystal_MS1V-T1K" (at 101.6 58.42 0)
+  (symbol (lib_id "power:PWR_FLAG") (at 64.77 86.36 0) (unit 1)
+    (in_bom yes) (on_board yes) (dnp no)
+    (property "Reference" "#FLG0101" (at 64.77 84.455 0)
+      (effects (font (size 1.27 1.27)) hide)
+    )
+    (property "Value" "PWR_FLAG" (at 64.77 81.9658 0)
+      (effects (font (size 1.27 1.27)))
+    )
+    (property "Footprint" "" (at 64.77 86.36 0)
+      (effects (font (size 1.27 1.27)) hide)
+    )
+    (property "Datasheet" "~" (at 64.77 86.36 0)
+      (effects (font (size 1.27 1.27)) hide)
+    )
+    (pin "1")
+    (instances
+      (project "Game_Cat_R4"
+        (path "/96315415-cfed-47d2-b3dd-d782358bd0df/00000000-0000-0000-0000-00005ce5bb47"
+          (reference "#FLG0101") (unit 1)
+        )
+      )
+    )
+  )
+  (symbol (lib_id "Device:Crystal_GND24") (at 101.6 58.42 90) (mirror x) (unit 1)
+    (in_bom yes) (on_board yes) (dnp no)
+    (property "Reference" "Y3" (at 90.17 58.42 90)
+      (effects (font (size 1.27 1.27)))
+    )
+    (property "Value" "ABS25" (at 91.44 60.96 90)
+      (effects (font (size 1.27 1.27)))
+    )
+    (property "Footprint" "x_Crystal:Crystal_SMD_Abracon_ABS25-4Pin_8.0x3.8mm" (at 101.6 58.42 0)
       (effects (font (size 1.27 1.27)) hide)
     )
@@
     (pin "1")
     (pin "2")
-    (instances
-      (project "Game_Cat_R4"
-        (path "/96315415-cfed-47d2-b3dd-d782358bd0df/00000000-0000-0000-0000-00005ce5bb47"
-          (reference "Y2") (unit 1)
-        )
-      )
-    )
-  )
-  (symbol (lib_id "power:PWR_FLAG") (at 64.77 86.36 0) (unit 1)
-    (in_bom yes) (on_board yes) (dnp no)
-    (property "Reference" "#FLG0101" (at 64.77 84.455 0)
-      (effects (font (size 1.27 1.27)) hide)
-    )
-    (property "Value" "PWR_FLAG" (at 64.77 81.9658 0)
-      (effects (font (size 1.27 1.27)))
-    )
-    (property "Footprint" "" (at 64.77 86.36 0)
-      (effects (font (size 1.27 1.27)) hide)
-    )
-    (property "Datasheet" "~" (at 64.77 86.36 0)
-      (effects (font (size 1.27 1.27)) hide)
-    )
-    (pin "1")
-    (instances
-      (project "Game_Cat_R4"
-        (path "/96315415-cfed-47d2-b3dd-d782358bd0df/00000000-0000-0000-0000-00005ce5bb47"
-          (reference "#FLG0101") (unit 1)
-        )
-      )
+    (pin "3")
+    (pin "4")
+    (instances
+      (project "STRANDING_ALPHA"
+        (path "/08da8f18-02c3-4a28-a400-670f01755980/00000000-0000-0000-0000-00005dfd13b7"
+          (reference "Y3") (unit 1)
+        )
+      )
+      (project "Game_Cat_R4"
+        (path "/96315415-cfed-47d2-b3dd-d782358bd0df/00000000-0000-0000-0000-00005ce5bb47"
+          (reference "Y3") (unit 1)
+        )
+      )

Commit message: 08/06/24/A
Parts:
- removed Y3: ABS25, x_Crystal:Crystal_SMD_Abracon_ABS25-4Pin_8.0x3.8mm, symbol Device:Crystal_GND24
- added Y2: Crystal_GND3, x_Crystal:MS1V-T1K_32.768KHZ_7PF_20PPM_TA, symbol Device:Crystal_GND3
Connections:
- net GND: now also Y2.3
- net at C9.2, U1.1 (PA00/XIN32): now also Y2.2
- net at C8.2, U1.2 (PA01/XOUT32): now also Y2.1
- no-connect marks 2 -> 0

Commit message: 25/01/24/A
Parts:
- added R63: 0R, Resistor_SMD:R_1206_3216Metric, symbol Device:R
- C12: value 10uF -> 1uF
Connections:
- net +3V3: now also R63.1; no longer L1.1
- net SCL: now also U1.26 (PA17); no longer U1.25 (PA16)
- net SDA: now also U1.25 (PA16); no longer U1.26 (PA17)
- new net: L1.1, R63.2
Changed lines of the file:
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@@
 	(wire
 		(pts
+			(xy 30.48 86.36) (xy 30.48 90.17)
+		)
+		(stroke
+			(width 0)
+			(type default)
+		)
+	)
+	(wire
+		(pts
 			(xy 181.61 85.09) (xy 208.28 85.09)
 		)
@@
 	(wire
 		(pts
+			(xy 30.48 74.93) (xy 30.48 78.74)
+		)
+		(stroke
+			(width 0)
+			(type default)
+		)
+	)
+	(wire
+		(pts
 			(xy 149.86 60.96) (xy 149.86 57.15)
 		)
@@
 	(wire
 		(pts
-			(xy 31.75 90.17) (xy 35.56 90.17)
+			(xy 30.48 90.17) (xy 35.56 90.17)
 		)
 		(stroke
@@
 	(wire
 		(pts
-			(xy 31.75 87.63) (xy 31.75 90.17)
-		)
-		(stroke
-			(width 0)
-			(type default)
-		)
-	)
-	(wire
-		(pts
 			(xy 101.6 81.28) (xy 115.57 81.28)
 		)
@@
 	(global_label "SDA"
 		(shape bidirectional)
-		(at 208.28 105.41 0)
+		(at 208.28 107.95 0)
 		(fields_autoplaced yes)
 		(effects
@@
 		)
 		(property "Intersheetrefs" "${INTERSHEET_REFS}"
-			(at 0 0 0)
+			(at 0 2.54 0)
 			(effects
 				(font
@@
 	(global_label "SCL"
 		(shape output)
-		(at 208.28 107.95 0)
+		(at 208.28 105.41 0)
 		(fields_autoplaced yes)
 		(effects
@@
 		)
 		(property "Intersheetrefs" "${INTERSHEET_REFS}"
-			(at 0 0 0)
+			(at 0 -2.54 0)
 			(effects
 				(font
@@
 	(symbol
 		(lib_id "power:+3.3V")
-		(at 31.75 87.63 0)
+		(at 30.48 74.93 0)
 		(unit 1)
 		(exclude_from_sim no)
@@
 		(dnp no)
 		(property "Reference" "#PWR01"
-			(at 31.75 91.44 0)
+			(at 30.48 78.74 0)
 			(effects
 				(font
@@
 		)
 		(property "Value" "+3V3"
-			(at 32.131 83.2358 0)
+			(at 30.861 70.5358 0)
 			(effects
 				(font
@@
 		)
 		(property "Footprint" ""
-			(at 31.75 87.63 0)
+			(at 30.48 74.93 0)
 			(effects
 				(font
@@
 		)
 		(property "Datasheet" ""
-			(at 31.75 87.63 0)
+			(at 30.48 74.93 0)
 			(effects
 				(font
@@
 		)
 		(property "Description" ""
-			(at 31.75 87.63 0)
+			(at 30.48 74.93 0)
 			(effects
 				(font
@@
 			)
 		)
-		(property "Value" "10uF"
+		(property "Value" "1uF"
 			(at 152.4 34.29 0)
 			(effects
@@
 			)
 		)
-		(property "Datasheet" ""
+		(property "Datasheet" "https://ww1.microchip.com/downloads/en/DeviceDoc/SAM-D21-DA1-Family-Data-Sheet-DS40001882H.pdf"
 			(at 156.21 101.6 0)
 			(effects
@@
 		)
 		(instances
-			(project "Game_Cat_R4"
+			(project ""
+				(path "/96315415-cfed-47d2-b3dd-d782358bd0df/00000000-0000-0000-0000-00005cbab8ae"
+					(reference "U1")
+					(unit 1)
+				)
 				(path "/96315415-cfed-47d2-b3dd-d782358bd0df/00000000-0000-0000-0000-00005ce5bb47"
 					(reference "U1")
@@
 					(unit 1)
 				)
+			)
+		)
+	)
+	(symbol
+		(lib_id "Device:R")
+		(at 30.48 82.55 0)
+		(mirror y)
+		(unit 1)
+		(exclude_from_sim no)
+		(in_bom yes)
+		(on_board yes)
+		(dnp no)
+		(property "Reference" "R63"
+			(at 28.702 81.3816 0)
+			(effects
+				(font
+					(size 1.27 1.27)
+				)
+				(justify left)
+			)
+		)
+		(property "Value" "0R"
+			(at 28.702 83.693 0)
+			(effects
+				(font
+					(size 1.27 1.27)
+				)
+				(justify left)
+			)
+		)
+		(property "Footprint" "Resistor_SMD:R_1206_3216Metric"
+			(at 32.258 82.55 90)
+			(effects
+				(font
+					(size 1.27 1.27)
+				)
+				(hide yes)
+			)
+		)
+		(property "Datasheet" "~"
+			(at 30.48 82.55 0)
+			(effects
+				(font
+					(size 1.27 1.27)
+				)
+				(hide yes)
+			)
+		)
+		(property "Description" ""
+			(at 30.48 82.55 0)
+			(effects
+				(font
+					(size 1.27 1.27)
+				)
+				(hide yes)
+			)
+		)
+		(pin "1"
+		)
+		(pin "2"
+		)
+		(instances
+			(project "Game_Cat_R4"
+				(path "/96315415-cfed-47d2-b3dd-d782358bd0df/00000000-0000-0000-0000-00005ce5bb47"
+					(reference "R63")
+					(unit 1)
+				)

Commit message: 05/25/25/A
Changed lines of the file:
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@@
 (kicad_sch
-	(version 20231120)
+	(version 20250114)
 	(generator "eeschema")
-	(generator_version "8.0")
+	(generator_version "9.0")
 	(paper "USLetter")
 	(title_block

Commit message: 03/11/26/Update BOM & Models VRML
Parts:
- C1: value 10uF -> 4.7uF; Digikey (none) -> TAJA475K016RNJ
- C12: Digikey (none) -> TAJA105K016RNJ
- C13, C2, C5: Digikey (none) -> C3216X7R2E104K160AE
- C8, C9: Digikey (none) -> C0805C220J5GAC7800
- L1: value BLM18PG471 -> FB321611T; Digikey (none) -> FB321611T-260Y-S
- R63: Digikey (none) -> RC1206FR-0710KL
- U1: Digikey (none) -> ATSAMD21G18A-AU
- Y2: footprint x_Crystal:MS1V-T1K_32.768KHZ_7PF_20PPM_TA -> x_Crystal:MS1V_T1K_32.768KHZ_7PF_20PPM_TA; Digikey (none) -> MS1V-T1K-32.768KHZ-9PF-20PPM-TA-QC
Changed lines of the file:
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@@
 			)
 		)
-		(property "Value" "BLM18PG471"
+		(property "Value" "FB321611T"
 			(at 41.91 87.63 90)
 			(effects
@@
 			)
 		)
-		(property "Datasheet" "~"
+		(property "Datasheet" "https://calchip.com/wp-content/uploads/2023/03/fb_series.pdf"
 			(at 39.37 90.17 0)
 			(effects
@@
 		(property "Description" ""
 			(at 39.37 90.17 0)
+			(effects
+				(font
+					(size 1.27 1.27)
+				)
+				(hide yes)
+			)
+		)
+		(property "Digikey" "FB321611T-260Y-S"
+			(at 39.37 90.17 90)
 			(effects
 				(font
@@
 			)
 		)
-		(property "Datasheet" "~"
+		(property "Datasheet" "https://product.tdk.com/system/files/dam/doc/product/capacitor/ceramic/mlcc/catalog/mlcc_commercial_soft_en.pdf"
 			(at 55.88 96.52 0)
 			(effects
@@
 		)
 		(property "Description" ""
+			(at 55.88 96.52 0)
+			(effects
+				(font
+					(size 1.27 1.27)
+				)
+				(hide yes)
+			)
+		)
+		(property "Digikey" "C3216X7R2E104K160AE"
 			(at 55.88 96.52 0)
 			(effects
@@
 			)
 		)
-		(property "Value" "10uF"
+		(property "Value" "4.7uF"
 			(at 48.641 97.663 0)
 			(effects
@@
 			)
 		)
-		(property "Datasheet" "~"
+		(property "Datasheet" "https://datasheets.kyocera-avx.com/TAJ.pdf"
 			(at 45.72 96.52 0)
 			(effects
@@
 		)
 		(property "Description" ""
+			(at 45.72 96.52 0)
+			(effects
+				(font
+					(size 1.27 1.27)
+				)
+				(hide yes)
+			)
+		)
+		(property "Digikey" "TAJA475K016RNJ"
 			(at 45.72 96.52 0)
 			(effects
@@
 			)
 		)
-		(property "Datasheet" "~"
+		(property "Datasheet" "https://product.tdk.com/system/files/dam/doc/product/capacitor/ceramic/mlcc/catalog/mlcc_commercial_soft_en.pdf"
 			(at 144.78 31.75 0)
 			(effects
@@
 		)
 		(property "Description" ""
+			(at 144.78 31.75 0)
+			(effects
+				(font
+					(size 1.27 1.27)
+				)
+				(hide yes)
+			)
+		)
+		(property "Digikey" "C3216X7R2E104K160AE"
 			(at 144.78 31.75 0)
 			(effects
@@
 			)
 		)
-		(property "Datasheet" "~"
+		(property "Datasheet" "https://datasheets.kyocera-avx.com/TAJ.pdf"
 			(at 149.86 31.75 0)
 			(effects
@@
 		)
 		(property "Description" ""
+			(at 149.86 31.75 0)
+			(effects
+				(font
+					(size 1.27 1.27)
+				)
+				(hide yes)
+			)
+		)
+		(property "Digikey" "TAJA105K016RNJ"
 			(at 149.86 31.75 0)
 			(effects
@@
 			)
 		)
-		(property "Datasheet" "~"
+		(property "Datasheet" "https://product.tdk.com/system/files/dam/doc/product/capacitor/ceramic/mlcc/catalog/mlcc_commercial_soft_en.pdf"
 			(at 185.42 71.12 0)
 			(effects
@@
 		)
 		(property "Description" ""
+			(at 185.42 71.12 0)
+			(effects
+				(font
+					(size 1.27 1.27)
+				)
+				(hide yes)
+			)
+		)
+		(property "Digikey" "C3216X7R2E104K160AE"
 			(at 185.42 71.12 0)
 			(effects
@@
 			)
 		)
-		(property "Description" ""
+		(property "Description" "ARM® Cortex®-M0+ SAM D21G, Functional Safety (FuSa) Microcontroller IC 32-Bit 48MHz 256KB (256K x 8) FLASH 48-TQFP (7x7)"
+			(at 148.59 93.98 0)
+			(effects
+				(font
+					(size 1.27 1.27)
+				)
+				(hide yes)
+			)
+		)
+		(property "Digikey" "ATSAMD21G18A-AU"
 			(at 148.59 93.98 0)
 			(effects
@@
 			)
 		)
-		(property "Datasheet" "~"
+		(property "Datasheet" "https://content.kemet.com/datasheets/KEM_C1003_C0G_SMD.pdf"
 			(at 96.52 64.77 0)
 			(effects
@@
 		(property "Description" ""
 			(at 96.52 64.77 0)
+			(effects
+				(font
+					(size 1.27 1.27)
+				)
+				(hide yes)
+			)
+		)
+		(property "Digikey" "C0805C220J5GAC7800"
+			(at 96.52 64.77 90)
 			(effects
 				(font
@@
 			)
 		)
-		(property "Datasheet" "~"
+		(property "Datasheet" "https://content.kemet.com/datasheets/KEM_C1003_C0G_SMD.pdf"
 			(at 96.52 52.07 0)
 			(effects
@@
 		(property "Description" ""
 			(at 96.52 52.07 0)
+			(effects
+				(font
+					(size 1.27 1.27)
+				)
+				(hide yes)
+			)
+		)
+		(property "Digikey" "C0805C220J5GAC7800"
+			(at 96.52 52.07 90)
 			(effects
 				(font
@@
 			)
 		)
-		(property "Footprint" "x_Crystal:MS1V-T1K_32.768KHZ_7PF_20PPM_TA"
+		(property "Footprint" "x_Crystal:MS1V_T1K_32.768KHZ_7PF_20PPM_TA"
 			(at 101.6 58.42 0)
 			(effects
@@
 			)
 		)
-		(property "Datasheet" "~"
+		(property "Datasheet" "https://www.microcrystal.com/fileadmin/Media/Products/32kHz/Datasheet/MS1V-T1K.pdf"
 			(at 101.6 58.42 0)
 			(effects
@@
 		(property "Description" "Three pin crystal, GND on pin 3"
 			(at 101.6 58.42 0)
+			(effects
+				(font
+					(size 1.27 1.27)
+				)
+				(hide yes)
+			)
+		)
+		(property "Digikey" "MS1V-T1K-32.768KHZ-9PF-20PPM-TA-QC"
+			(at 101.6 58.42 90)
 			(effects
 				(font
@@
 			)
 		)
-		(property "Datasheet" "~"
+		(property "Datasheet" "https://www.yageogroup.com/content/datasheet/asset/file/PYU-RC_GROUP_51_ROHS_L"
 			(at 30.48 82.55 0)
 			(effects
@@
 			(at 30.48 82.55 0)
 			(effects
+				(font
+					(size 1.27 1.27)
+				)
+				(hide yes)
+			)
+		)
+		(property "Digikey" "RC1206FR-0710KL"
+			(at 30.48 82.55 0)
+			(effects
