File: power_supply.kicad_sch (KiCad schematic)
At the start: 56 parts, among them J5 CORTEX-SWD, J7 PWM, Q4 DMP3056L, Q5 NTR1P02LT1, Q8 BS138, Q9 BS138, SW7 Reset, SW8 SW_SPDT, U11 MCP73831, U12 TPS54231

Commit message: 25/01/24/A
Parts:
- removed R4: 1K, Resistor_SMD:R_1206_3216Metric, symbol Device:R
- added D10: BAT60J, Diode_SMD:D_SOD-323_HandSoldering, symbol Device:D_Schottky
- added Q11: IRFL901, Package_TO_SOT_SMD:SOT-223-3_TabPin2, symbol Device:Q_PMOS_GDS
- added R64: 0R, Resistor_SMD:R_1206_3216Metric, symbol Device:R
- C36: value 4.7uF -> 1uF
- R37: value 68K -> 30K
- R40: value 1K -> 180
- R43: value 68K -> 3K
Connections:
- net +3V3: now also D10.1 (K), R64.1; no longer C42.1, L3.2, R42.1
- net RESET: now also D10.2 (A)
- new net: C42.1, L3.2, R42.1, R64.2
Other:
- moved on the sheet: R38, TP14

Commit message: 25/01/24/C
Parts:
- removed Q11: IRFL901, Package_TO_SOT_SMD:SOT-223-3_TabPin2, symbol Device:Q_PMOS_GDS
Changed lines of the file:
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@@
-	)
-	(symbol
-		(lib_id "Device:Q_PMOS_GDS")
-		(at 115.57 20.32 270)
-		(unit 1)
-		(exclude_from_sim no)
-		(in_bom yes)
-		(on_board yes)
-		(dnp no)
-		(property "Reference" "Q11"
-			(at 115.57 26.67 90)
-			(effects
-				(font
-					(size 1.27 1.27)
-				)
-			)
-		)
-		(property "Value" "IRFL901"
-			(at 115.57 29.21 90)
-			(effects
-				(font
-					(size 1.27 1.27)
-				)
-			)
-		)
-		(property "Footprint" "Package_TO_SOT_SMD:SOT-223-3_TabPin2"
-			(at 118.11 25.4 0)
-			(effects
-				(font
-					(size 1.27 1.27)
-				)
-				(hide yes)
-			)
-		)
-		(property "Datasheet" "~"
-			(at 115.57 20.32 0)
-			(effects
-				(font
-					(size 1.27 1.27)
-				)
-				(hide yes)
-			)
-		)
-		(property "Description" ""
-			(at 115.57 20.32 0)
-			(effects
-				(font
-					(size 1.27 1.27)
-				)
-				(hide yes)
-			)
-		)
-		(pin "1"
-		)
-		(pin "2"
-		)
-		(pin "3"
-		)
-		(instances
-			(project "Game_Cat_R4"
-				(path "/96315415-cfed-47d2-b3dd-d782358bd0df/00000000-0000-0000-0000-00005ccc9b26"
-					(reference "Q11")
-					(unit 1)
-				)
-			)
-		)
 	)
 	(symbol

Commit message: 25/01/26/A
Parts:
- removed D7: BAT60J, Diode_SMD:D_SOD-323_HandSoldering, symbol Device:D_Schottky
Changed lines of the file:
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@@
 	)
 	(junction
-		(at 116.84 67.31)
-		(diameter 0)
-		(color 0 0 0 0)
-	)
-	(junction
 		(at 139.7 113.03)
 		(diameter 0)
@@
 	(wire
 		(pts
-			(xy 116.84 64.77) (xy 116.84 67.31)
-		)
-		(stroke
-			(width 0)
-			(type default)
-		)
-	)
-	(wire
-		(pts
 			(xy 184.15 64.77) (xy 186.69 64.77)
 		)
@@
 	(wire
 		(pts
-			(xy 116.84 57.15) (xy 116.84 55.88)
-		)
-		(stroke
-			(width 0)
-			(type default)
-		)
-	)
-	(wire
-		(pts
 			(xy 90.17 102.87) (xy 53.34 102.87)
 		)
@@
 	(wire
 		(pts
-			(xy 116.84 67.31) (xy 125.73 67.31)
+			(xy 115.57 67.31) (xy 125.73 67.31)
 		)
 		(stroke
@@
 	(wire
 		(pts
-			(xy 116.84 67.31) (xy 115.57 67.31)
-		)
-		(stroke
-			(width 0)
-			(type default)
-		)
-	)
-	(wire
-		(pts
 			(xy 139.7 121.92) (xy 139.7 123.19)
 		)
@@
 	)
 	(label "BRG"
-		(at 125.73 45.72 0)
-		(fields_autoplaced yes)
+		(at 124.46 45.72 0)
 		(effects
 			(font
@@
 	(label "M"
 		(at 110.49 55.88 0)
-		(fields_autoplaced yes)
 		(effects
 			(font
@@
 	(label "ON-OFF"
 		(at 104.14 67.31 0)
-		(fields_autoplaced yes)
 		(effects
 			(font
@@
 	(label "PROG"
 		(at 72.39 48.26 0)
-		(fields_autoplaced yes)
 		(effects
 			(font
@@
 	(label "+BATT"
 		(at 104.14 45.72 0)
-		(fields_autoplaced yes)
 		(effects
 			(font
@@
 	(label "BAT_L"
 		(at 45.72 50.8 0)
-		(fields_autoplaced yes)
 		(effects
 			(font
@@
 					(unit 1)
 				)
-			)
-		)
-	)
-	(symbol
-		(lib_id "Device:D_Schottky")
-		(at 116.84 60.96 270)
-		(unit 1)
-		(exclude_from_sim no)
-		(in_bom yes)
-		(on_board yes)
-		(dnp no)
-		(property "Reference" "D7"
-			(at 114.8334 62.1284 90)
-			(effects
-				(font
-					(size 1.27 1.27)
-				)
-				(justify right)
-			)
-		)
-		(property "Value" "BAT60J"
-			(at 124.46 64.77 90)
-			(effects
-				(font
-					(size 1.27 1.27)
-				)
-				(justify right)
-			)
-		)
-		(property "Footprint" "Diode_SMD:D_SOD-323_HandSoldering"
-			(at 116.84 60.96 0)
-			(effects
-				(font
-					(size 1.27 1.27)
-				)
-				(hide yes)
-			)
-		)
-		(property "Datasheet" "~"
-			(at 116.84 60.96 0)
-			(effects
-				(font
-					(size 1.27 1.27)
-				)
-				(hide yes)
-			)
-		)
-		(property "Description" ""
-			(at 116.84 60.96 0)
-			(effects
-				(font
-					(size 1.27 1.27)
-				)
-				(hide yes)
-			)
-		)
-		(pin "1"
-		)
-		(pin "2"
-		)
-		(instances
-			(project "Game_Cat_R4"
-				(path "/96315415-cfed-47d2-b3dd-d782358bd0df/00000000-0000-0000-0000-00005ccc9b26"
-					(reference "D7")
-					(unit 1)
-				)

Commit message: 05/25/25/A
Parts:
- removed C43, C44: 100nF, Capacitor_SMD:C_1206_3216Metric, symbol Device:C
- Q4: value DMP3056L -> FDN340P

Commit message: 03/11/26/Update BOM & Models VRML
Parts:
- BT1: footprint x_Connector_JST:Connector_1x02_P2.0mm -> x_Connector_JST:S2B_PH_SM4_TB
- C33, C40: Digikey (none) -> C3216X7R2E104K160AE
- C36, C45: Digikey (none) -> TAJA105K016RNJ
- C37: Digikey (none) -> GRM21A5C2E470JW01D
- C38: Digikey (none) -> GCM31A5C3A150FX01D
- C39: Digikey (none) -> TAJA475K016RNJ
- C41: Digikey (none) -> GRM3195C1H113JA01D
- C42: Digikey (none) -> GCM31A5C3A470FX01D
- D10, D8: Digikey (none) -> BAT60JFILM
- D4, D5: footprint LED_SMD:LED_0805_2012Metric_Castellated -> LED_SMD:LED_0805_2012Metric; Digikey (none) -> LTST-C170GKT
- D9: Digikey (none) -> LTST-C170GKT
- L3: Digikey (none) -> 82103C
- Q4: Digikey (none) -> FDN340P
- Q5: Digikey (none) -> NTR1P02LT1G
- Q8, Q9: value BS138 -> BSS138; Digikey (none) -> BSS138
- R30, R31, R32, R39, R41, R42, R50, R51, R52, R53, R62, R64: Digikey (none) -> RC1206FR-0710KL
- R33, R34: Digikey (none) -> RC1206JR-07470RL
- R35: Digikey (none) -> RC1206FR-07332RL
- R36: Digikey (none) -> RC1206FR-0768KL
- R37: Digikey (none) -> RC1206FR-0730KL
- R38, R44: Digikey (none) -> RC1206FR-072KL
- R40: Digikey (none) -> RC1206JR-07180RL
- R43: Digikey (none) -> RC1206FR-073KL
- R49: Digikey (none) -> RC1206JR-0733RL
- SW7: Digikey (none) -> PTS645SK50SMTR92 LFS
- TP11, TP12, TP13, TP14, TP29: now not fitted
- U11: Digikey (none) -> MCP73831T-5ACI/OT
- U12: Digikey (none) -> TPS54231D

Commit message: 03/12/26/Update BOM & Models VRML
Parts:
- BT1: Digikey (none) -> S2B-PH-SM4-TB
- D6: Digikey (none) -> 1N5819HWQ-7-F
- J5: Digikey (none) -> 61200621721
- J7: Digikey (none) -> SWR25X-NRTC-S04-RB-BA
- SW8: Digikey (none) -> PCM12SMTR
Changed lines of the file:
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@@
 			)
 		)
-		(property "Datasheet" "~"
+		(property "Datasheet" "https://www.jst-mfg.com/product/pdf/eng/ePH.pdf"
 			(at 95.25 59.436 90)
 			(effects
@@
 			)
 		)
-		(property "Description" ""
+		(property "Description" "CONN HEADER SMD R/A 2POS 2MM"
+			(at 95.25 60.96 0)
+			(effects
+				(font
+					(size 1.27 1.27)
+				)
+				(hide yes)
+			)
+		)
+		(property "Digikey" "S2B-PH-SM4-TB"
 			(at 95.25 60.96 0)
 			(effects
@@
 			)
 		)
-		(property "Datasheet" "~"
+		(property "Datasheet" "https://www.ckswitches.com/media/1424/pcm.pdf"
 			(at 110.49 69.85 0)
 			(effects
@@
 			)
 		)
+		(property "Digikey" "PCM12SMTR"
+			(at 110.49 69.85 0)
+			(effects
+				(font
+					(size 1.27 1.27)
+				)
+				(hide yes)
+			)
+		)
 		(pin "1"
 		)
@@
 			)
 		)
-		(property "Datasheet" "~"
+		(property "Datasheet" "https://www.diodes.com/assets/Datasheets/1N5819HWQ.pdf"
 			(at 118.11 118.11 0)
 			(effects
@@
 			)
 		)
+		(property "Digikey" "1N5819HWQ-7-F"
+			(at 118.11 118.11 90)
+			(effects
+				(font
+					(size 1.27 1.27)
+				)
+				(hide yes)
+			)
+		)
 		(pin "1"
 		)
@@
 			)
 		)
-		(property "Datasheet" "~"
+		(property "Datasheet" "https://mm.digikey.com/Volume0/opasdata/d220001/medias/docus/386/SWR25X-NRTC-Sxx-Rx-BA.pdf"
 			(at 245.11 109.22 0)
 			(effects
@@
 			)
 		)
-		(property "Description" ""
+		(property "Description" "CONN HEADER R/A 4POS 2.54MM"
+			(at 245.11 109.22 0)
+			(effects
+				(font
+					(size 1.27 1.27)
+				)
+				(hide yes)
+			)
+		)
+		(property "Digikey" "SWR25X-NRTC-S04-RB-BA"
 			(at 245.11 109.22 0)
 			(effects
@@
 			)
 		)
-		(property "Datasheet" "~"
+		(property "Datasheet" "https://www.we-online.com/components/products/datasheet/61200621721.pdf"
 			(at 34.29 176.53 0)
 			(effects
@@
 			)
 		)
-		(property "Description" ""
+		(property "Description" "CONN HEADER R/A 6POS 2.54MM"
+			(at 34.29 176.53 0)
+			(effects
+				(font
+					(size 1.27 1.27)
+				)
+				(hide yes)
+			)
+		)
+		(property "Digikey" "61200621721"
 			(at 34.29 176.53 0)
 			(effects
